File: Pi-ic880a.sch (EAGLE design)
At the start: 28 parts, among them U1 IC880A, U2 BR24G32-3, U3 DS3231SN

Commit message: After adding all other GPIO
Connections:
- new net !GPS_RESET: PI1.IO27, U1.!GPS_RESET
- new net EN_GPS: PI1.IO23, U1.EN_GPS
- new net SP_VALID: PI1.IO24, U1.SP_VALID
- new net SX1301_GPIO0: PI1.SPI1_SCLK, U1.SX1301GPIO0
- new net SX1301_GPIO1: PI1.SPI1_MOSI, U1.SX1301GPIO1
- new net SX1301_GPIO2: PI1.IO12, U1.SX1301GPIO2
- new net SX1301_GPIO3: PI1.IO16, U1.SX1301GPIO3
- new net SX1301_GPIO4: PI1.IO5, U1.SX1301GPIO4
- net SX1301_RST: now also PI1.IO17; no longer PI1.IO27
Changed lines of the file:
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@@
 <segment>
 <pinref part="PI1" gate="G$1" pin="IO6"/>
-<wire x1="55.88" y1="208.28" x2="36.83" y2="208.28" width="0.1524" layer="91"/>
-<label x="36.83" y="208.28" size="1.778" layer="95"/>
+<wire x1="55.88" y1="208.28" x2="31.75" y2="208.28" width="0.1524" layer="91"/>
+<label x="31.75" y="208.28" size="1.778" layer="95"/>
 </segment>
 </net>
@@
 <segment>
 <pinref part="PI1" gate="G$1" pin="SPI0_SCLK"/>
-<wire x1="55.88" y1="218.44" x2="35.56" y2="218.44" width="0.1524" layer="91"/>
-<label x="36.83" y="218.44" size="1.778" layer="95"/>
+<wire x1="55.88" y1="218.44" x2="31.75" y2="218.44" width="0.1524" layer="91"/>
+<label x="31.75" y="218.44" size="1.778" layer="95"/>
 </segment>
 </net>
@@
 <segment>
 <pinref part="PI1" gate="G$1" pin="SPI0_MISO"/>
-<wire x1="55.88" y1="220.98" x2="35.56" y2="220.98" width="0.1524" layer="91"/>
-<label x="36.83" y="220.98" size="1.778" layer="95"/>
+<wire x1="55.88" y1="220.98" x2="31.75" y2="220.98" width="0.1524" layer="91"/>
+<label x="31.75" y="220.98" size="1.778" layer="95"/>
 </segment>
 </net>
@@
 <segment>
 <pinref part="PI1" gate="G$1" pin="SPI0_MOSI"/>
-<wire x1="55.88" y1="223.52" x2="35.56" y2="223.52" width="0.1524" layer="91"/>
-<label x="36.83" y="223.52" size="1.778" layer="95"/>
+<wire x1="55.88" y1="223.52" x2="31.75" y2="223.52" width="0.1524" layer="91"/>
+<label x="31.75" y="223.52" size="1.778" layer="95"/>
 </segment>
 </net>
@@
 <segment>
 <pinref part="PI1" gate="G$1" pin="SPI0_CS0"/>
-<wire x1="99.06" y1="218.44" x2="119.38" y2="218.44" width="0.1524" layer="91"/>
-<label x="106.68" y="218.44" size="1.778" layer="95"/>
+<wire x1="99.06" y1="218.44" x2="124.46" y2="218.44" width="0.1524" layer="91"/>
+<label x="105.41" y="218.44" size="1.778" layer="95"/>
 </segment>
 </net>
@@
 <segment>
 <pinref part="PI1" gate="G$1" pin="ID_SC"/>
-<wire x1="99.06" y1="213.36" x2="119.38" y2="213.36" width="0.1524" layer="91"/>
-<label x="106.68" y="213.36" size="1.778" layer="95"/>
+<wire x1="99.06" y1="213.36" x2="124.46" y2="213.36" width="0.1524" layer="91"/>
+<label x="105.41" y="213.36" size="1.778" layer="95"/>
 </segment>
 </net>
@@
 <segment>
 <pinref part="PI1" gate="G$1" pin="ID_SD"/>
-<wire x1="55.88" y1="213.36" x2="35.56" y2="213.36" width="0.1524" layer="91"/>
-<label x="36.83" y="213.36" size="1.778" layer="95"/>
+<wire x1="55.88" y1="213.36" x2="31.75" y2="213.36" width="0.1524" layer="91"/>
+<label x="31.75" y="213.36" size="1.778" layer="95"/>
 </segment>
 </net>
@@
 <segment>
 <pinref part="PI1" gate="G$1" pin="I2C1_SDA"/>
-<wire x1="55.88" y1="243.84" x2="36.83" y2="243.84" width="0.1524" layer="91"/>
-<label x="36.83" y="243.84" size="1.778" layer="95"/>
+<wire x1="55.88" y1="243.84" x2="31.75" y2="243.84" width="0.1524" layer="91"/>
+<label x="31.75" y="243.84" size="1.778" layer="95"/>
 </segment>
 <segment>
@@
 <segment>
 <pinref part="PI1" gate="G$1" pin="I2C1_SCL"/>
-<wire x1="55.88" y1="241.3" x2="36.83" y2="241.3" width="0.1524" layer="91"/>
-<label x="36.83" y="241.3" size="1.778" layer="95"/>
+<wire x1="55.88" y1="241.3" x2="31.75" y2="241.3" width="0.1524" layer="91"/>
+<label x="31.75" y="241.3" size="1.778" layer="95"/>
 </segment>
 <segment>
@@
 <segment>
 <pinref part="PI1" gate="G$1" pin="TXD"/>
-<wire x1="99.06" y1="238.76" x2="116.84" y2="238.76" width="0.1524" layer="91"/>
-<label x="106.68" y="238.76" size="1.778" layer="95"/>
+<wire x1="99.06" y1="238.76" x2="124.46" y2="238.76" width="0.1524" layer="91"/>
+<label x="105.41" y="238.76" size="1.778" layer="95"/>
 </segment>
 </net>
@@
 <segment>
 <pinref part="PI1" gate="G$1" pin="RXD"/>
-<wire x1="99.06" y1="236.22" x2="116.84" y2="236.22" width="0.1524" layer="91"/>
-<label x="106.68" y="236.22" size="1.778" layer="95"/>
+<wire x1="99.06" y1="236.22" x2="124.46" y2="236.22" width="0.1524" layer="91"/>
+<label x="105.41" y="236.22" size="1.778" layer="95"/>
 </segment>
 </net>
@@
 <segment>
 <pinref part="PI1" gate="G$1" pin="IO22"/>
-<wire x1="55.88" y1="228.6" x2="36.83" y2="228.6" width="0.1524" layer="91"/>
-<label x="36.83" y="228.6" size="1.778" layer="95"/>
+<wire x1="55.88" y1="228.6" x2="31.75" y2="228.6" width="0.1524" layer="91"/>
+<label x="31.75" y="228.6" size="1.778" layer="95"/>
 </segment>
 </net>
@@
 </segment>
 <segment>
-<pinref part="PI1" gate="G$1" pin="IO27"/>
-<wire x1="55.88" y1="231.14" x2="36.83" y2="231.14" width="0.1524" layer="91"/>
-<label x="36.83" y="231.14" size="1.778" layer="95"/>
+<pinref part="PI1" gate="G$1" pin="IO17"/>
+<wire x1="55.88" y1="233.68" x2="31.75" y2="233.68" width="0.1524" layer="91"/>
+<label x="31.75" y="233.68" size="1.778" layer="95"/>
 </segment>
 </net>
@@
 </segment>
 </net>
+<net name="EN_GPS" class="0">
+<segment>
+<pinref part="U1" gate="G$1" pin="EN_GPS"/>
+<wire x1="274.32" y1="208.28" x2="256.54" y2="208.28" width="0.1524" layer="91"/>
+<label x="256.54" y="208.28" size="1.778" layer="95"/>
+</segment>
+<segment>
+<pinref part="PI1" gate="G$1" pin="IO23"/>
+<wire x1="99.06" y1="228.6" x2="124.46" y2="228.6" width="0.1524" layer="91"/>
+<label x="105.41" y="228.6" size="1.778" layer="95"/>
+</segment>
+</net>
+<net name="!GPS_RESET" class="0">
+<segment>
+<pinref part="U1" gate="G$1" pin="!GPS_RESET"/>
+<wire x1="274.32" y1="205.74" x2="256.54" y2="205.74" width="0.1524" layer="91"/>
+<label x="256.54" y="205.74" size="1.778" layer="95"/>
+</segment>
+<segment>
+<pinref part="PI1" gate="G$1" pin="IO27"/>
+<wire x1="55.88" y1="231.14" x2="31.75" y2="231.14" width="0.1524" layer="91"/>
+<label x="31.75" y="231.14" size="1.778" layer="95"/>
+</segment>
+</net>
+<net name="SX1301_GPIO0" class="0">
+<segment>
+<pinref part="U1" gate="G$1" pin="SX1301GPIO0"/>
+<wire x1="320.04" y1="220.98" x2="337.82" y2="220.98" width="0.1524" layer="91"/>
+<label x="325.12" y="220.98" size="1.778" layer="95"/>
+</segment>
+<segment>
+<pinref part="PI1" gate="G$1" pin="SPI1_SCLK"/>
+<wire x1="99.06" y1="198.12" x2="124.46" y2="198.12" width="0.1524" layer="91"/>
+<label x="105.41" y="198.12" size="1.778" layer="95"/>
+</segment>
+</net>
+<net name="SX1301_GPIO1" class="0">
+<segment>
+<pinref part="U1" gate="G$1" pin="SX1301GPIO1"/>
+<wire x1="320.04" y1="218.44" x2="337.82" y2="218.44" width="0.1524" layer="91"/>
+<label x="325.12" y="218.44" size="1.778" layer="95"/>
+</segment>
+<segment>
+<pinref part="PI1" gate="G$1" pin="SPI1_MOSI"/>
+<wire x1="99.06" y1="200.66" x2="124.46" y2="200.66" width="0.1524" layer="91"/>
+<label x="105.41" y="200.66" size="1.778" layer="95"/>
+</segment>
+</net>
+<net name="SX1301_GPIO2" class="0">
+<segment>
+<pinref part="U1" gate="G$1" pin="SX1301GPIO2"/>
+<wire x1="320.04" y1="215.9" x2="337.82" y2="215.9" width="0.1524" layer="91"/>
+<label x="325.12" y="215.9" size="1.778" layer="95"/>
+</segment>
+<segment>
+<pinref part="PI1" gate="G$1" pin="IO12"/>
+<wire x1="99.06" y1="208.28" x2="124.46" y2="208.28" width="0.1524" layer="91"/>
+<label x="105.41" y="208.28" size="1.778" layer="95"/>
+</segment>
+</net>
+<net name="SX1301_GPIO3" class="0">
+<segment>
+<pinref part="U1" gate="G$1" pin="SX1301GPIO3"/>
+<wire x1="320.04" y1="213.36" x2="337.82" y2="213.36" width="0.1524" layer="91"/>
+<label x="325.12" y="213.36" size="1.778" layer="95"/>
+</segment>
+<segment>
+<pinref part="PI1" gate="G$1" pin="IO16"/>
+<wire x1="99.06" y1="203.2" x2="124.46" y2="203.2" width="0.1524" layer="91"/>
+<label x="105.41" y="203.2" size="1.778" layer="95"/>
+</segment>
+</net>
+<net name="SX1301_GPIO4" class="0">
+<segment>
+<pinref part="U1" gate="G$1" pin="SX1301GPIO4"/>
+<wire x1="320.04" y1="210.82" x2="337.82" y2="210.82" width="0.1524" layer="91"/>
+<label x="325.12" y="210.82" size="1.778" layer="95"/>
+</segment>
+<segment>
+<pinref part="PI1" gate="G$1" pin="IO5"/>
+<wire x1="55.88" y1="210.82" x2="31.75" y2="210.82" width="0.1524" layer="91"/>
+<label x="31.75" y="210.82" size="1.778" layer="95"/>
+</segment>
+</net>
+<net name="SP_VALID" class="0">
+<segment>
+<pinref part="U1" gate="G$1" pin="SP_VALID"/>
+<wire x1="320.04" y1="195.58" x2="337.82" y2="195.58" width="0.1524" layer="91"/>
+<label x="325.12" y="195.58" size="1.778" layer="95"/>
+</segment>
+<segment>
+<pinref part="PI1" gate="G$1" pin="IO24"/>
+<wire x1="99.06" y1="226.06" x2="124.46" y2="226.06" width="0.1524" layer="91"/>
+<label x="105.41" y="226.06" size="1.778" layer="95"/>
+</segment>
+</net>
