File: Pi-ic880a.sch (EAGLE design)
At the start: 28 parts, among them U1 IC880A, U2 BR24G32-3, U3 DS3231SN

Commit message: V2 about ready to go
Parts:
- C3: value 100pf -> 100nf
Changed lines of the file:
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@@
 <?xml version="1.0" encoding="utf-8"?>
 <!DOCTYPE eagle SYSTEM "eagle.dtd">
-<eagle version="8.4.1">
+<eagle version="8.4.2">
 <drawing>
 <settings>
@@
 <part name="+3V2" library="supply1" library_urn="urn:adsk.eagle:library:371" deviceset="+3V3" device=""/>
 <part name="U$3" library="fruit-parts" deviceset="TEMP-HUM-SENSOR-DHT22" device=""/>
-<part name="C3" library="Seeed-Capacitor" library_urn="urn:adsk.eagle:library:464" deviceset="CERAMIC-100PF-50V-5%-NPO(0603)" device="" package3d_urn="urn:adsk.eagle:package:32378/1" value="100pf"/>
+<part name="C3" library="Seeed-Capacitor" library_urn="urn:adsk.eagle:library:464" deviceset="CERAMIC-100PF-50V-5%-NPO(0603)" device="" package3d_urn="urn:adsk.eagle:package:32378/1" value="100nf"/>
 <part name="R6" library="Seeed-Resistor" library_urn="urn:adsk.eagle:library:474" deviceset="SMD-RES-10K-1%-1/10W(0603)" device="" package3d_urn="urn:adsk.eagle:package:32791/1" value="10K"/>
 <part name="+3V6" library="supply1" library_urn="urn:adsk.eagle:library:371" deviceset="+3V3" device=""/>

Commit message: DC jack added Now called Pi-CoT smd GPS moved closer to ant holes for Pi connector now bigger
Parts:
- added J1: FC681465P, farnell-parts:FC681465P
Connections:
- net +5V: now also J1.+
- net GND: now also J1.-
Other:
- note added: "DC in"
Changed lines of the file:
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@@
 <part name="R9" library="Seeed-Resistor" library_urn="urn:adsk.eagle:library:474" deviceset="SMD-RES-0R-5%-1/10W(0603)" device="" package3d_urn="urn:adsk.eagle:package:32791/1" value="0R"/>
 <part name="TP3" library="testpad" library_urn="urn:adsk.eagle:library:385" deviceset="TP" device="B2,54" package3d_urn="urn:adsk.eagle:package:27948/1"/>
+<part name="J1" library="farnell-parts" deviceset="FC681465P" device=""/>
+<part name="GND12" library="supply1" library_urn="urn:adsk.eagle:library:371" deviceset="GND" device=""/>
+<part name="P+3" library="supply1" library_urn="urn:adsk.eagle:library:371" deviceset="+5V" device=""/>
 </parts>
 <sheets>
@@
 <wire x1="151.13" y1="177.8" x2="3.81" y2="177.8" width="0.1524" layer="150"/>
 <text x="40.64" y="81.28" size="6.4516" layer="97">Onboard GPS</text>
+<text x="179.07" y="154.94" size="6.4516" layer="150">DC in</text>
 </plain>
 <instances>
@@
 <instance part="R9" gate="G$1" x="181.61" y="106.68"/>
 <instance part="TP3" gate="G$1" x="194.31" y="119.38"/>
+<instance part="J1" gate="G$1" x="186.69" y="179.07"/>
+<instance part="GND12" gate="1" x="193.04" y="173.99"/>
+<instance part="P+3" gate="1" x="203.2" y="185.42"/>
 </instances>
 <busses>
@@
 <wire x1="99.06" y1="246.38" x2="99.06" y2="250.19" width="0.1524" layer="91"/>
 <junction x="99.06" y="246.38"/>
+</segment>
+<segment>
+<pinref part="J1" gate="G$1" pin="+"/>
+<pinref part="P+3" gate="1" pin="+5V"/>
+<wire x1="193.04" y1="181.61" x2="203.2" y2="181.61" width="0.1524" layer="91"/>
+<wire x1="203.2" y1="181.61" x2="203.2" y2="182.88" width="0.1524" layer="91"/>
 </segment>
 </net>
@@
 <junction x="184.15" y="227.33"/>
 </segment>
+<segment>
+<pinref part="J1" gate="G$1" pin="-"/>
+<pinref part="GND12" gate="1" pin="GND"/>
+</segment>
 </net>
